File: module-fast-imaging/strobe_pcb/strobe-pcb.sch (EAGLE design)
At the start: 7 parts, among them IC2 PIC16F18857

Commit message: First strobe PCB submitted.
Parts:
- added R3: (no value), rcl:R-EU_R1206
- added R4: (no value), rcl:R-EU_0207/10
Connections:
- net N$10 renamed SPI_IN
- net N$11 renamed STROBE_GATE
- net N$13 renamed SPI_SS
- net N$15 renamed STROBE_TRIG_IN
- net N$3 renamed SPI_OUT
- net N$4 renamed SPI_CLOCK
- net N$5 renamed SPI_MCLR
- net N$9 renamed ISCP_PGD
- net V_HIGH renamed STROBE-
- new net +12V: IC1.14, R4.1
- new net +5V: IC1.13
- new net STROBE+_RES: IC1.15, R4.2
- new net STROBE_0V: IC1.18, Q1.S, R3.1
- net GND: no longer IC1.18, Q1.S
- net N$12: now also R3.2
Other:
- moved on the sheet: IC1, Q1

Commit message: Added resistor.
Connections:
- net ISCP_PGD renamed ICSP_PGD
- net SPI_CLOCK renamed SPI_CLK
- net SPI_MCLR renamed ICSP_MCLR
Changed lines of the file:
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@@
 </segment>
 </net>
-<net name="SPI_CLOCK" class="0">
+<net name="SPI_CLK" class="0">
 <segment>
 <pinref part="IC1" gate="G$1" pin="26"/>
@@
 </segment>
 </net>
-<net name="SPI_MCLR" class="0">
+<net name="ICSP_MCLR" class="0">
 <segment>
 <pinref part="IC2" gate="G$1" pin="!MCLR/THV"/>
@@
 </segment>
 </net>
-<net name="ISCP_PGD" class="0">
+<net name="ICSP_PGD" class="0">
 <segment>
 <pinref part="IC2" gate="G$1" pin="PGD/RB7"/>
