File: module-fast-imaging/strobe_pcb/strobe-pcb.brd (EAGLE design)
At the start: 36 x 19 mm, 7 parts, among them IC2 PIC16F18857

Commit message: First strobe PCB submitted.
Parts:
- added R3: (no value), rcl:R1206
- added R4: (no value), rcl:0207/10
- moved R2 2.51 mm to (42.8, 27.5)
Connections:
- net N$10 renamed SPI_IN
- net N$11 renamed STROBE_GATE
- net N$13 renamed SPI_SS
- net N$15 renamed STROBE_TRIG_IN
- net N$3 renamed SPI_OUT
- net N$4 renamed SPI_CLOCK
- net N$5 renamed SPI_MCLR
- net N$9 renamed ISCP_PGD
- net V_HIGH renamed STROBE-
- new net +12V: IC1.14, R4.1
- new net +5V: IC1.13
- new net STROBE+_RES: IC1.15, R4.2
- new net STROBE_0V: IC1.18, Q1.S, R3.1
- net GND: no longer IC1.18, Q1.S
- net N$12: now also R3.2
Routing:
- net STROBE+_RES: track 0.00 -> 22.6 mm
- net +12V: track 0.00 -> 14.2 mm
- net STROBE_0V: track 0.00 -> 12.6 mm
- net GND: track 19.6 -> 10.8 mm, vias 3 -> 5
- net N$12: track 4.59 -> 9.52 mm
- net STROBE_GATE: track 27.8 -> 31.0 mm

Commit message: Added resistor.
Connections:
- net ISCP_PGD renamed ICSP_PGD
- net SPI_CLOCK renamed SPI_CLK
- net SPI_MCLR renamed ICSP_MCLR
Changed lines of the file:
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@@
 <wire x1="13.49" y1="36.182" x2="13.5" y2="36.172" width="0.254" layer="16"/>
 </signal>
-<signal name="SPI_CLOCK">
+<signal name="SPI_CLK">
 <contactref element="IC1" pad="26"/>
 <contactref element="IC2" pad="24"/>
@@
 <wire x1="19.46" y1="37.54" x2="18.57" y2="38.43" width="0.254" layer="1"/>
 </signal>
-<signal name="SPI_MCLR">
+<signal name="ICSP_MCLR">
 <contactref element="IC2" pad="1"/>
 <contactref element="IC1" pad="1"/>
@@
 <wire x1="23.65" y1="26.1" x2="23.65" y2="23.38" width="0.254" layer="16"/>
 </signal>
-<signal name="ISCP_PGD">
+<signal name="ICSP_PGD">
 <contactref element="IC2" pad="28"/>
 <contactref element="IC1" pad="4"/>

Commit message: PICkit3 profiles.
Parts:
- C1: value (none) -> 100nf
- C2: value (none) -> 1uf
- R1: value (none) -> 1k
- R2: value (none) -> 510
- R3: value (none) -> 10k
Changed lines of the file:
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@@
 <attribute name="VALUE" x="46.58" y="39.62" size="1.27" layer="27" ratio="10" rot="R180"/>
 </element>
-<element name="C1" library="rcl" library_urn="urn:adsk.eagle:library:334" package="C1206" package3d_urn="urn:adsk.eagle:package:23618/2" value="" x="25" y="36" smashed="yes" rot="MR180">
+<element name="C1" library="rcl" library_urn="urn:adsk.eagle:library:334" package="C1206" package3d_urn="urn:adsk.eagle:package:23618/2" value="100nf" x="25" y="36" smashed="yes" rot="MR180">
 <attribute name="NAME" x="27.73" y="36.73" size="1.27" layer="26" rot="MR180"/>
 <attribute name="SPICEPREFIX" value="C" x="25" y="36" size="1.778" layer="28" rot="MR180" display="off"/>
 <attribute name="VALUE" x="23.73" y="38.54" size="1.27" layer="28" rot="MR180"/>
 </element>
-<element name="C2" library="rcl" library_urn="urn:adsk.eagle:library:334" package="C1206" package3d_urn="urn:adsk.eagle:package:23618/2" value="" x="25" y="33.75" smashed="yes" rot="MR180">
+<element name="C2" library="rcl" library_urn="urn:adsk.eagle:library:334" package="C1206" package3d_urn="urn:adsk.eagle:package:23618/2" value="1uf" x="25" y="33.75" smashed="yes" rot="MR180">
 <attribute name="NAME" x="27.73" y="34.48" size="1.27" layer="26" rot="MR180"/>
 <attribute name="SPICEPREFIX" value="C" x="25" y="33.75" size="1.778" layer="28" rot="MR180" display="off"/>
 <attribute name="VALUE" x="23.73" y="36.29" size="1.27" layer="28" rot="MR180"/>
 </element>
-<element name="R1" library="rcl" library_urn="urn:adsk.eagle:library:334" package="R1206" package3d_urn="urn:adsk.eagle:package:23540/2" value="" x="13.5" y="34.75" smashed="yes" rot="MR270">
+<element name="R1" library="rcl" library_urn="urn:adsk.eagle:library:334" package="R1206" package3d_urn="urn:adsk.eagle:package:23540/2" value="1k" x="13.5" y="34.75" smashed="yes" rot="MR270">
 <attribute name="NAME" x="14.73" y="34.48" size="1.27" layer="26" rot="MR180"/>
 <attribute name="POPULARITY" value="41" x="13.5" y="34.75" size="1.778" layer="28" rot="MR270" display="off"/>
@@
 <attribute name="VALUE" x="16.04" y="36.02" size="1.27" layer="28" rot="MR270"/>
 </element>
-<element name="R2" library="rcl" library_urn="urn:adsk.eagle:library:334" package="R1206" package3d_urn="urn:adsk.eagle:package:23540/2" value="" x="42.75" y="27.5" smashed="yes" rot="R180">
+<element name="R2" library="rcl" library_urn="urn:adsk.eagle:library:334" package="R1206" package3d_urn="urn:adsk.eagle:package:23540/2" value="510" x="42.75" y="27.5" smashed="yes" rot="R180">
 <attribute name="NAME" x="44.02" y="26.23" size="1.27" layer="25" rot="R180"/>
 <attribute name="POPULARITY" value="41" x="42.75" y="27.5" size="1.778" layer="27" rot="R180" display="off"/>
@@
 <attribute name="VALUE" x="44.02" y="30.04" size="1.27" layer="27" rot="R180"/>
 </element>
-<element name="R3" library="rcl" library_urn="urn:adsk.eagle:library:334" package="R1206" package3d_urn="urn:adsk.eagle:package:23540/2" value="" x="40.5" y="30.25" smashed="yes">
+<element name="R3" library="rcl" library_urn="urn:adsk.eagle:library:334" package="R1206" package3d_urn="urn:adsk.eagle:package:23540/2" value="10k" x="40.5" y="30.25" smashed="yes">
 <attribute name="NAME" x="39.23" y="31.52" size="1.27" layer="25"/>
 <attribute name="POPULARITY" value="41" x="40.5" y="30.25" size="1.778" layer="27" display="off"/>
