File: module-sample-holders/sample_holder_pcb/sample-holder-pcb.brd (EAGLE design)
At the start: 36 x 36 mm, 35 parts, among them IC1 25AA040ST, IC2 DSPIC33CK256MP502-I_SS, Q1 AUIRFU8403

Commit message: PCB documentation.
Parts:
- C7: value (none) -> Unfitted
- T1, T3: value (none) -> NPN
- T2, T4: value (none) -> PNP
Changed lines of the file:
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@@
 <?xml version="1.0" encoding="utf-8"?>
 <!DOCTYPE eagle SYSTEM "eagle.dtd">
-<eagle version="9.5.1">
+<eagle version="9.5.2">
 <drawing>
 <settings>
@@
 <setting verticaltext="up"/>
 </settings>
-<grid distance="0.25" unitdist="mm" unit="mm" style="lines" multiple="1" display="yes" altdistance="0.125" altunitdist="mm" altunit="mm"/>
+<grid distance="0.25" unitdist="mm" unit="mm" style="lines" multiple="1" display="no" altdistance="0.125" altunitdist="mm" altunit="mm"/>
 <layers>
-<layer number="1" name="Top" color="4" fill="1" visible="no" active="yes"/>
+<layer number="1" name="Top" color="4" fill="1" visible="yes" active="yes"/>
 <layer number="2" name="Route2" color="1" fill="3" visible="no" active="no"/>
 <layer number="3" name="Route3" color="4" fill="3" visible="no" active="no"/>
@@
 <attribute name="VALUE" x="45.25" y="28.425" size="1.27" layer="27" rot="R180"/>
 </element>
-<element name="T1" library="transistor" library_urn="urn:adsk.eagle:library:402" package="SOT23-BEC" package3d_urn="urn:adsk.eagle:package:28748/2" value="" x="25" y="40.25" smashed="yes" rot="R180">
+<element name="T1" library="transistor" library_urn="urn:adsk.eagle:library:402" package="SOT23-BEC" package3d_urn="urn:adsk.eagle:package:28748/2" value="NPN" x="25" y="40.25" smashed="yes" rot="R180">
 <attribute name="NAME" x="23.905" y="42.845" size="1.27" layer="25" rot="R180"/>
 <attribute name="POPULARITY" value="0" x="25" y="40.25" size="1.778" layer="27" rot="R180" display="off"/>
 <attribute name="VALUE" x="26.905" y="43.425" size="1.27" layer="27" rot="R180"/>
 </element>
-<element name="T2" library="transistor" library_urn="urn:adsk.eagle:library:402" package="SOT23-BEC" package3d_urn="urn:adsk.eagle:package:28748/2" value="" x="28" y="40" smashed="yes" rot="MR90">
+<element name="T2" library="transistor" library_urn="urn:adsk.eagle:library:402" package="SOT23-BEC" package3d_urn="urn:adsk.eagle:package:28748/2" value="PNP" x="28" y="40" smashed="yes" rot="MR90">
 <attribute name="NAME" x="24.655" y="38.845" size="1.27" layer="26" rot="MR90"/>
 <attribute name="POPULARITY" value="0" x="28" y="40" size="1.778" layer="28" rot="MR90" display="off"/>
@@
 <attribute name="VALUE" x="42.255" y="47.19" size="1.27" layer="27" rot="R90"/>
 </element>
-<element name="T3" library="transistor" library_urn="urn:adsk.eagle:library:402" package="SOT23-BEC" package3d_urn="urn:adsk.eagle:package:28748/2" value="" x="22" y="38.25" smashed="yes" rot="R90">
+<element name="T3" library="transistor" library_urn="urn:adsk.eagle:library:402" package="SOT23-BEC" package3d_urn="urn:adsk.eagle:package:28748/2" value="NPN" x="22" y="38.25" smashed="yes" rot="R90">
 <attribute name="NAME" x="22.155" y="40.095" size="1.27" layer="25" rot="R180"/>
 <attribute name="POPULARITY" value="0" x="22" y="38.25" size="1.778" layer="27" rot="R90" display="off"/>
@@
 <attribute name="VALUE" x="22.405" y="35.615" size="1.27" layer="27" rot="R90"/>
 </element>
-<element name="T4" library="transistor" library_urn="urn:adsk.eagle:library:402" package="SOT23-BEC" package3d_urn="urn:adsk.eagle:package:28748/2" value="" x="22.125" y="33.375" smashed="yes" rot="R270">
+<element name="T4" library="transistor" library_urn="urn:adsk.eagle:library:402" package="SOT23-BEC" package3d_urn="urn:adsk.eagle:package:28748/2" value="PNP" x="22.125" y="33.375" smashed="yes" rot="R270">
 <attribute name="NAME" x="21.97" y="31.28" size="1.27" layer="25"/>
 <attribute name="POPULARITY" value="0" x="22.125" y="33.375" size="1.778" layer="27" rot="R270" display="off"/>
@@
 <attribute name="VALUE" x="43.095" y="34.115" size="1.27" layer="28" rot="MR90"/>
 </element>
-<element name="C7" library="rcl" library_urn="urn:adsk.eagle:library:334" package="C0603" package3d_urn="urn:adsk.eagle:package:23616/2" value="" x="41" y="35.5" smashed="yes" rot="MR90">
+<element name="C7" library="rcl" library_urn="urn:adsk.eagle:library:334" package="C0603" package3d_urn="urn:adsk.eagle:package:23616/2" value="Unfitted" x="41" y="35.5" smashed="yes" rot="MR90">
 <attribute name="NAME" x="38.885" y="34.365" size="1.27" layer="26" rot="MR90"/>
 <attribute name="SPICEPREFIX" value="C" x="41" y="35.5" size="1.778" layer="28" rot="MR90" display="off"/>
